File: USB_C_PSU.kicad_sch (KiCad schematic)
At the start: 97 parts, among them J101 BATTERY, J102 I2C, J103 USB_C, J104 PWR, J105 DATA1, Q101 BSH205G2A, Q102 DMP6050SSD, Q103 2N7002H, SW101 SW_SPDT, U101 TPS63070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

Commit message: pdf and readme file
Other:
- note added: "3.3V Buck-Boost Converter"
- note removed: "3.3V Switching Regulator"
- note removed: "Current needs VCC -> 3v3 converter in: - MCU: 128mA max - DAC/ Mux stuff: ~5mA - LED (x65): 16mA max - Display: ~30mA (guess) - Total: 1198mA - Should equate to ~850 mA at 5V converter input assuming claimed 93% efficiency - Or 1417mA at 3V converter input VCC -> 12V converter in: - TL07x (x218): 1.6 mA (348mA) - LM13700 (x12): 2.6mA (31.2mA) - TOTAL: 380mA - About 1072mA from 5V assuming 85% eff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"
- moved on the sheet: C101, C102, C103, C104, C105, C107, C108, C111, D108, J102, J104, J105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

Commit message: finished readme
Other:
- note added: "R106 sets the constant charging current at ~300mA (p. 14 of the datasheet)"
- note removed: "R704 sets the constant charging current at ~300mA (p. 14 of the datasheet)"
Changed lines of the file:
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@@
 		)
 	)
-	(text "R704 sets the constant\ncharging current at ~300mA\n(p. 14 of the datasheet)"
+	(text "R106 sets the constant\ncharging current at ~300mA\n(p. 14 of the datasheet)"
 		(exclude_from_sim no)
 		(at 215.646 81.788 0)
